File: PHASEB/Board__Micro/BoardMicro.kicad_pcb (KiCad board)
At the start: 2 copper layers, 68.6 x 53.3 mm, 20 parts, among them J1 Power, J2 Digital/PWM, J3 Analog, J4 Digital/PWM, J5 CONN_GYRO, J6 CONN_DISPLAY, J7 CONN_TEMP, SW1 SW_SPST, SW2 SW_SPST, SW3 SW_SPST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

Commit message: Add files via upload
Parts:
- added G***: LOGO, LOGO, F.Cu at (115.0, 97.0)
Routing:
- net GND: track 119.4 -> 123.8 mm, vias 9 -> 8
- net /button_units: track 36.1 -> 35.0 mm
- net /button_lock: track 50.1 -> 49.1 mm
- net /button_onoff: track 77.3 -> 76.4 mm
- net /button_light: track 71.3 -> 72.1 mm
- net /button_cal: track 63.7 -> 62.8 mm
- net /I2C_SDA: track 28.9 -> 28.4 mm
- net /I2C_SCL: track 27.6 -> 27.1 mm
Other:
- board text added: "Button ON/OFF"
- board text added: "Button Units"
- board text added: "Calibration"
- board text added: "LED"
- board text added: "Light Button"
- board text added: "Lock Button"
- board text added: "Temp Sensor"
- board text added: "Version 1 2/3/2025 Alexis Romo"
